Commit message: pcl filter, lake fix. pointcloud-based corridor construction ready

File: gazebo_sim/urdf/intersection_lane.urdf (robot description, URDF)
Before this commit: robot simple_box, 1 links, 0 joints
Links:
- link my_box: geometry collision box size=10 0.3 1.0; visual box size=10 0.3 1.0

File: gazebo_sim/urdf/lane.urdf (robot description, URDF)
Before this commit: robot simple_box, 1 links, 0 joints
Links:
- link my_box: geometry collision box size=15 0.3 1.0; visual box size=15 0.3 1.0

File: gazebo_sim/urdf/long_lane.urdf (robot description, URDF)
Before this commit: robot simple_box, 1 links, 0 joints
Links:
- link my_box: geometry collision box size=22.4 0.3 1.0; visual box size=22.4 0.3 1.0
